Commit message: add changes from this morning see if errror occurs

File: 41068_ignition_bringup/urdf_drone/parrot.urdf.xacro (robot description, xacro)
@@ -124,3 +124,28 @@
   </joint>
   <link name="camera_depth_optical_frame"/>
+  <!-- Thermal camera link mounted off the main camera boom -->
+  <joint name="thermal_camera_joint" type="fixed">
+    <!-- offset from camera_link: 5 cm down, rotated to look down -->
+    <origin xyz="0 0 -0.05" rpy="0 1.57 0"/>
+    <parent link="camera_link"/>
+    <child link="thermal_camera_link"/>
+  </joint>
+  <link name="thermal_camera_link">
+    <!-- tiny visual just so we can see it in Gazebo/rviz if needed -->
+    <visual>
+      <origin xyz="0 0 0" rpy="0 0 0"/>
+      <geometry>
+        <box size="0.02 0.02 0.02"/>
+      </geometry>
+      <material name="dark"/>
+    </visual>
+    <!-- light inertial so URDF is happy -->
+    <inertial>
+      <origin xyz="0 0 0" rpy="0 0 0"/>
+      <mass value="0.001"/>
+      <inertia ixx="1e-6" ixy="0" ixz="0"
+               iyy="1e-6" iyz="0"
+               izz="1e-6"/>
+    </inertial>
+  </link>
 </robot>

Commit message: build but no image on thermal camera

File: 41068_ignition_bringup/urdf_drone/parrot.urdf.xacro (robot description, xacro)
@@ -126,9 +126,8 @@
   <!-- Thermal camera link mounted off the main camera boom -->
   <joint name="thermal_camera_joint" type="fixed">
-    <joint name="thermal_camera_joint" type="fixed">
-      <origin xyz="0 0 0" rpy="0 0.785398 0"/>
-      <parent link="camera_link"/>
-      <child link="thermal_camera_link"/>
-    </joint>
+    <origin xyz="0 0 0" rpy="0 0.785398 0"/>
+    <parent link="camera_link"/>
+    <child link="thermal_camera_link"/>
+  </joint>
   <link name="thermal_camera_link">
     <!-- tiny visual just so we can see it in Gazebo/rviz if needed -->
