Commit message: Thermal Cam Setup test

File: 41068_ignition_bringup/urdf_drone/parrot.gazebo.xacro (robot description, xacro)
@@ -169,16 +169,13 @@
       <gz_frame_id>camera_link</gz_frame_id>
     </sensor>
-    <!-- new thermal camera on the same link -->
+  </gazebo>
+  <gazebo reference="thermal_camera_link">
     <sensor name="thermal_camera" type="thermal">
-      <!-- 5 cm below the camera, pitched down 90 deg -->
-      <pose>0 0 -0.05 0 1.57 0</pose>
-      <always_on>true</always_on>
-      <update_rate>10</update_rate>
-      <visualize>true</visualize>
-      <thermal_camera>
+      <camera>
+        <horizontal_fov>1.047</horizontal_fov>
         <image>
           <width>320</width>
           <height>240</height>
-          <format>L16</format>
+          <format>L8</format>   <!-- L8 = 8 Bit, L16 = 16 bit thermal cam -->
         </image>
         <clip>
@@ -186,7 +183,17 @@
           <far>20</far>
         </clip>
-      </thermal_camera>
+      </camera>
+      <always_on>1</always_on>
+      <update_rate>30</update_rate>
+      <visualize>true</visualize>
       <topic>/model/parrot/thermal_camera/image</topic>
-      <gz_frame_id>camera_link</gz_frame_id>
+      <gz_frame_id>thermal_camera_link</gz_frame_id>
+      <plugin
+        filename="ignition-gazebo-thermal-sensor-system"
+        name="gz::sim::systems::ThermalSensor">
+        <min_temp>253.15</min_temp>   <!-- -20C -->
+        <max_temp>773.15</max_temp>   <!-- 500C -->
+        <resolution>3.0</resolution>
+      </plugin>
     </sensor>
   </gazebo>

File: 41068_ignition_bringup/urdf_drone/parrot.urdf.xacro (robot description, xacro)
@@ -124,3 +124,28 @@
   </joint>
   <link name="camera_depth_optical_frame"/>
+    <!-- Thermal camera link mounted off the main camera boom -->
+  <joint name="thermal_camera_joint" type="fixed">
+    <!-- offset from camera_link: 5 cm down, rotated to look down -->
+    <origin xyz="0 0 -0.05" rpy="0 1.57 0"/>
+    <parent link="camera_link"/>
+    <child link="thermal_camera_link"/>
+  </joint>
+  <link name="thermal_camera_link">
+    <!-- tiny visual just so we can see it in Gazebo/rviz if needed -->
+    <visual>
+      <origin xyz="0 0 0" rpy="0 0 0"/>
+      <geometry>
+        <box size="0.02 0.02 0.02"/>
+      </geometry>
+      <material name="dark"/>
+    </visual>
+    <!-- light inertial so URDF is happy -->
+    <inertial>
+      <origin xyz="0 0 0" rpy="0 0 0"/>
+      <mass value="0.001"/>
+      <inertia ixx="1e-6" ixy="0" ixz="0"
+               iyy="1e-6" iyz="0"
+               izz="1e-6"/>
+    </inertial>
+  </link>
 </robot>

Commit message: ok if this doesnt fix it it isnt my fault

File: 41068_ignition_bringup/urdf_drone/parrot.gazebo.xacro (robot description, xacro)
@@ -169,13 +169,16 @@
       <gz_frame_id>camera_link</gz_frame_id>
     </sensor>
-  </gazebo>
-  <gazebo reference="thermal_camera_link">
+    <!-- new thermal camera on the same link -->
     <sensor name="thermal_camera" type="thermal">
-      <camera>
-        <horizontal_fov>1.047</horizontal_fov>
+      <!-- 5 cm below the camera, pitched down 90 deg -->
+      <pose>0 0 -0.05 0 1.57 0</pose>
+      <always_on>true</always_on>
+      <update_rate>10</update_rate>
+      <visualize>true</visualize>
+      <thermal_camera>
         <image>
           <width>320</width>
           <height>240</height>
-          <format>L8</format>   <!-- L8 = 8 Bit, L16 = 16 bit thermal cam -->
+          <format>L16</format>
         </image>
         <clip>
@@ -183,17 +186,7 @@
           <far>20</far>
         </clip>
-      </camera>
-      <always_on>1</always_on>
-      <update_rate>30</update_rate>
-      <visualize>true</visualize>
+      </thermal_camera>
       <topic>/model/parrot/thermal_camera/image</topic>
-      <gz_frame_id>thermal_camera_link</gz_frame_id>
-      <plugin
-        filename="ignition-gazebo-thermal-sensor-system"
-        name="gz::sim::systems::ThermalSensor">
-        <min_temp>253.15</min_temp>   <!-- -20C -->
-        <max_temp>773.15</max_temp>   <!-- 500C -->
-        <resolution>3.0</resolution>
-      </plugin>
+      <gz_frame_id>camera_link</gz_frame_id>
     </sensor>
   </gazebo>

File: 41068_ignition_bringup/urdf_drone/parrot.urdf.xacro (robot description, xacro)
@@ -124,28 +124,3 @@
   </joint>
   <link name="camera_depth_optical_frame"/>
-    <!-- Thermal camera link mounted off the main camera boom -->
-  <joint name="thermal_camera_joint" type="fixed">
-    <!-- offset from camera_link: 5 cm down, rotated to look down -->
-    <origin xyz="0 0 -0.05" rpy="0 1.57 0"/>
-    <parent link="camera_link"/>
-    <child link="thermal_camera_link"/>
-  </joint>
-  <link name="thermal_camera_link">
-    <!-- tiny visual just so we can see it in Gazebo/rviz if needed -->
-    <visual>
-      <origin xyz="0 0 0" rpy="0 0 0"/>
-      <geometry>
-        <box size="0.02 0.02 0.02"/>
-      </geometry>
-      <material name="dark"/>
-    </visual>
-    <!-- light inertial so URDF is happy -->
-    <inertial>
-      <origin xyz="0 0 0" rpy="0 0 0"/>
-      <mass value="0.001"/>
-      <inertia ixx="1e-6" ixy="0" ixz="0"
-               iyy="1e-6" iyz="0"
-               izz="1e-6"/>
-    </inertial>
-  </link>
 </robot>

Commit message: changed thermal view

File: 41068_ignition_bringup/urdf_drone/parrot.gazebo.xacro (robot description, xacro)
@@ -191,4 +191,5 @@
       <plugin filename="libignition-gazebo-thermal-sensor-system.so"
               name="ignition::gazebo::systems::ThermalSensor">
+        <render_engine>ogre2</render_engine>
         <min_temp>253.15</min_temp> <!-- 22C  -->
         <max_temp>773.15</max_temp> <!-- 500C -->
@@ -198,10 +199,2 @@
   </gazebo>
 </robot>
-<!-- TODO: find the right path to this plugin -->
-<!-- <plugin>
-        filename="ignition-gazebo-thermal-sensor-system.so"
-        name="gz::sim::systems::ThermalSensor"
-        <min_temp>253.15</min_temp>
-        <max_temp>773.15</max_temp>
-        <resolution>3.0</resolution>
-      </plugin> -->

File: 41068_ignition_bringup/urdf_drone/parrot.urdf.xacro (robot description, xacro)
@@ -126,9 +126,9 @@
   <!-- Thermal camera link mounted off the main camera boom -->
   <joint name="thermal_camera_joint" type="fixed">
-    <!-- offset from camera_link: 5 cm down, rotated to look down -->
-    <origin xyz="0 0 -0.05" rpy="0 1.57 0"/>
-    <parent link="camera_link"/>
-    <child link="thermal_camera_link"/>
-  </joint>
+    <joint name="thermal_camera_joint" type="fixed">
+      <origin xyz="0 0 0" rpy="0 0.785398 0"/>
+      <parent link="camera_link"/>
+      <child link="thermal_camera_link"/>
+    </joint>
   <link name="thermal_camera_link">
     <!-- tiny visual just so we can see it in Gazebo/rviz if needed -->

Commit message: Thermal cam now working visualising same FOV as camera and differentiating temp

File: 41068_ignition_bringup/urdf_drone/parrot.gazebo.xacro (robot description, xacro)
@@ -173,8 +173,8 @@
     <sensor name="thermal_camera" type="thermal">
       <camera>
-        <horizontal_fov>1.047</horizontal_fov>
+        <horizontal_fov>2.0944</horizontal_fov>
         <image>
-          <width>320</width>
-          <height>240</height>
+          <width>720</width>    <!-- originally 320 -->
+          <height>480</height>  <!-- originally 240 -->
           <format>L8</format>   <!-- L8 = 8 Bit, L16 = 16 bit thermal cam -->
         </image>

File: 41068_ignition_bringup/urdf_drone/parrot.urdf.xacro (robot description, xacro)
@@ -126,5 +126,5 @@
   <!-- Thermal camera link mounted off the main camera boom -->
   <joint name="thermal_camera_joint" type="fixed">
-    <origin xyz="0 0 0" rpy="0 0.785398 0"/>
+    <origin xyz="0 0 0" rpy="0 0 0"/>
     <parent link="camera_link"/>
     <child link="thermal_camera_link"/>

Commit message: depth camera rotated weirdly finding solution

File: 41068_ignition_bringup/urdf_drone/parrot.gazebo.xacro (robot description, xacro)
@@ -188,5 +188,5 @@
       <visualize>true</visualize>
       <topic>/model/parrot/thermal_camera/image</topic>
-      <gz_frame_id>thermal_camera_link</gz_frame_id>
+      <gz_frame_id>thermal_camera_optical_frame</gz_frame_id>
       <plugin filename="libignition-gazebo-thermal-sensor-system.so"
               name="ignition::gazebo::systems::ThermalSensor">

File: 41068_ignition_bringup/urdf_drone/parrot.urdf.xacro (robot description, xacro)
@@ -148,3 +148,9 @@
     </inertial>
   </link>
+  <joint name="thermal_camera_optical_joint" type="fixed">
+    <origin xyz="0 0 0" rpy="-1.57 0 -1.57"/>
+    <parent link="thermal_camera_link"/>
+    <child link="thermal_camera_optical_frame"/>
+  </joint>
+  <link name="thermal_camera_optical_frame"/>
 </robot>
