Commit message: Fixed reliance on 41068 package, neatened up mission package

File: pyrosens_ignition_bringup/urdf_drone/parrot.gazebo.xacro (robot description, xacro)
@@ -4,5 +4,5 @@
   <xacro:arg name="camera_visual" default="false"/>
   <xacro:arg name="imu_visual"    default="false"/>
-  <!-- <xacro:include filename="$(find 41068_ignition_bringup)/urdf/wheel.urdf.xacro"/> -->
+  <!-- <xacro:include filename="$(find pyrosens_ignition_bringup)/urdf/wheel.urdf.xacro"/> -->
   <gazebo reference="imu_link">
     <sensor type="imu" name="imu">

File: pyrosens_ignition_bringup/urdf_drone/parrot.urdf.xacro (robot description, xacro)
@@ -1,6 +1,6 @@
 <?xml version="1.0" ?>
 <robot name="parrot" xmlns:xacro="http://ros.org/wiki/xacro">
-  <xacro:include filename="$(find 41068_ignition_bringup)/urdf_drone/common_properties.urdf.xacro"/>
-  <xacro:include filename="$(find 41068_ignition_bringup)/urdf_drone/parrot.gazebo.xacro"/>
+  <xacro:include filename="$(find pyrosens_ignition_bringup)/urdf_drone/common_properties.urdf.xacro"/>
+  <xacro:include filename="$(find pyrosens_ignition_bringup)/urdf_drone/parrot.gazebo.xacro"/>
   <xacro:property name="r200_cam_rgb_px" value="0.005"/>
   <xacro:property name="r200_cam_rgb_py" value="0.018"/>
@@ -24,5 +24,5 @@
     <visual name="hull">
       <geometry>
-        <mesh filename="file://$(find 41068_ignition_bringup)/urdf_drone/meshes/hull.dae"/>
+        <mesh filename="file://$(find pyrosens_ignition_bringup)/urdf_drone/meshes/hull.dae"/>
       </geometry>
     </visual>
@@ -30,5 +30,5 @@
       <origin xyz="-0.09035 -0.11423 -0.00501" rpy="0 0 0"/>
       <geometry>
-        <mesh filename="file://$(find 41068_ignition_bringup)/urdf_drone/meshes/propeller_rr.dae"/>
+        <mesh filename="file://$(find pyrosens_ignition_bringup)/urdf_drone/meshes/propeller_rr.dae"/>
       </geometry>
     </visual>
@@ -36,5 +36,5 @@
       <origin xyz="0.09035 0.11452 -0.00501" rpy="0 0 0"/>
       <geometry>
-        <mesh filename="file://$(find 41068_ignition_bringup)/urdf_drone/meshes/propeller_rl.dae"/>
+        <mesh filename="file://$(find pyrosens_ignition_bringup)/urdf_drone/meshes/propeller_rl.dae"/>
       </geometry>
     </visual>
@@ -42,5 +42,5 @@
       <origin xyz="0.08456 -0.11435 -0.00501" rpy="0 0 0"/>
       <geometry>
-        <mesh filename="file://$(find 41068_ignition_bringup)/urdf_drone/meshes/propeller_fr.dae"/>
+        <mesh filename="file://$(find pyrosens_ignition_bringup)/urdf_drone/meshes/propeller_fr.dae"/>
       </geometry>
     </visual>
@@ -48,5 +48,5 @@
       <origin xyz="0.08456 0.11463 -0.00501" rpy="0 0 0"/>
       <geometry>
-        <mesh filename="file://$(find 41068_ignition_bringup)/urdf_drone/meshes/propeller_fl.dae"/>
+        <mesh filename="file://$(find pyrosens_ignition_bringup)/urdf_drone/meshes/propeller_fl.dae"/>
       </geometry>
     </visual>
